File: HSS/power-switch/anti-spark-pcb.sch (EAGLE design)
At the start: 9 parts

Commit message: laceration v3 some files
Parts:
- removed JP1: M01PTH, anti-spark-pcb:M01PTH
- removed R5: (no value), anti-spark-pcb:RESISTOR1206
- removed SJ1: (no value), anti-spark-pcb:SOLDERJUMPER_2WAYS
- R1: value 39R / RCS120639R0FKEA -> 39R / EP1WSSS39RJ; device anti-spark-pcb:RESISTOR1206 -> anti-spark-pcb:RESISTORPTH-1W
- R4: value (none) -> 0R
Connections:
- removed net N$8: R5.1, SJ1.2
- removed net N$9: JP1.1, R5.2
- net N$1: no longer SJ1.3
- net N$2: no longer SJ1.1
